Commit message: made some changes

File: examples/valkyrie/urdf/atlas_urdf/atlas_convex_hull.urdf (robot description, URDF)
Before this commit: robot atlas, 70 links, 69 joints
Links:
- link head: geometry collision mesh filename=package://valkyrie/urdf/meshes/head_chull.obj; visual mesh filename=package://valkyrie/urdf/meshes/head_chull.obj
- link hokuyo_link: geometry collision mesh filename=package://valkyrie/urdf/meshes/head_camera_chull.obj; visual mesh filename=package://valkyrie/urdf/meshes/head_camera_chull.obj
- link l_clav: geometry collision mesh filename=package://valkyrie/urdf/meshes/r_clav_chull.obj; visual mesh filename=package://valkyrie/urdf/atlas_urdfmeshes/r_clav.obj
- link l_foot: geometry collision mesh filename=package://valkyrie/urdf/meshes/l_foot_chull.obj; collision sphere radius=0.0
- link l_larm: geometry collision mesh filename=package://valkyrie/urdf/meshes/r_larm_chull.obj; visual mesh filename=package://valkyrie/urdf/meshes/r_larm.obj
- link l_lfarm: geometry collision mesh filename=package://valkyrie/urdf/meshes/r_hand_chull.obj; visual mesh filename=package://valkyrie/urdf/meshes/r_hand.obj
- link l_lglut: geometry collision mesh filename=package://valkyrie/urdf/meshes/l_lglut_chull.obj; visual mesh filename=package://valkyrie/urdf/meshes/l_lglut.obj
- link l_lleg: geometry collision mesh filename=package://valkyrie/urdf/meshes/l_lleg_chull.obj; visual mesh filename=package://valkyrie/urdf/meshes/l_lleg.obj
- link l_scap: geometry collision mesh filename=package://valkyrie/urdf/meshes/r_scap_chull.obj; visual mesh filename=package://valkyrie/urdf/meshes/r_scap.obj
- link l_talus: geometry visual mesh filename=package://valkyrie/urdf/meshes/l_talus.obj
- link l_uarm: geometry collision mesh filename=package://valkyrie/urdf/meshes/r_uarm_chull.obj; visual mesh filename=package://valkyrie/urdf/meshes/r_uarm.obj
- link l_ufarm: geometry collision mesh filename=package://valkyrie/urdf/meshes/r_farm_chull.obj; visual mesh filename=package://valkyrie/urdf/meshes/r_farm.obj
- link l_uglut: geometry collision mesh filename=package://valkyrie/urdf/meshes/l_uglut_chull.obj; visual mesh filename=package://valkyrie/urdf/meshes/l_uglut.obj
- link l_uleg: geometry collision mesh filename=package://valkyrie/urdf/meshes/l_uleg_chull.obj; visual mesh filename=package://valkyrie/urdf/meshes/l_uleg.obj
- link left_palm: geometry collision mesh filename=package://valkyrie/urdf/meshes/GRIPPER_OPEN_chull.obj scale=1 1 1; visual mesh filename=package://valkyrie/urdf/meshes/GRIPPER_OPEN_chull.obj scale=1 1 1
- link ltorso: geometry visual mesh filename=package://valkyrie/urdf/meshes/ltorso.obj
- link mtorso: geometry visual mesh filename=package://valkyrie/urdf/meshes/mtorso.obj
- link pelvis: geometry collision mesh filename=package://valkyrie/urdf/meshes/pelvis_chull.obj; visual mesh filename=package://valkyrie/urdf/meshes/pelvis.obj
- link r_clav: geometry collision mesh filename=package://valkyrie/urdf/meshes/r_clav_chull.obj; visual mesh filename=package://valkyrie/urdf/meshes/r_clav.obj
- link r_foot: geometry collision mesh filename=package://valkyrie/urdf/meshes/r_foot_chull.obj; collision sphere radius=0.0
- link r_larm: geometry collision mesh filename=package://valkyrie/urdf/meshes/r_larm_chull.obj; visual mesh filename=package://valkyrie/urdf/meshes/r_larm.obj
- link r_lfarm: geometry collision mesh filename=package://valkyrie/urdf/meshes/r_hand_chull.obj; visual mesh filename=package://valkyrie/urdf/meshes/r_hand.obj
- link r_lglut: geometry collision mesh filename=package://valkyrie/urdf/meshes/r_lglut_chull.obj; visual mesh filename=package://valkyrie/urdf/meshes/r_lglut.obj
- link r_lleg: geometry collision mesh filename=package://valkyrie/urdf/meshes/r_lleg_chull.obj; visual mesh filename=package://valkyrie/urdf/meshes/r_lleg.obj
- link r_scap: geometry collision mesh filename=package://valkyrie/urdf/meshes/r_scap_chull.obj; visual mesh filename=package://valkyrie/urdf/meshes/r_scap.obj
- link r_talus: geometry visual mesh filename=package://valkyrie/urdf/meshes/r_talus.obj
- link r_uarm: geometry collision mesh filename=package://valkyrie/urdf/meshes/r_uarm_chull.obj; visual mesh filename=package://valkyrie/urdf/meshes/r_uarm.obj
- link r_ufarm: geometry collision mesh filename=package://valkyrie/urdf/meshes/r_farm_chull.obj; visual mesh filename=package://valkyrie/urdf/meshes/r_farm.obj
- link r_uglut: geometry collision mesh filename=package://valkyrie/urdf/meshes/r_uglut_chull.obj; visual mesh filename=package://valkyrie/urdf/meshes/r_uglut.obj
- link r_uleg: geometry collision mesh filename=package://valkyrie/urdf/meshes/r_uleg_chull.obj; visual mesh filename=package://valkyrie/urdf/meshes/r_uleg.obj
- link right_palm: geometry collision mesh filename=package://valkyrie/urdf/meshes/GRIPPER_OPEN_chull.obj scale=1 1 1; visual mesh filename=package://valkyrie/urdf/meshes/GRIPPER_OPEN_chull.obj scale=1 1 1
- link utorso: geometry collision mesh filename=package://valkyrie/urdf/meshes/utorso_chull.obj; visual mesh filename=package://valkyrie/urdf/meshes/utorso.obj

Commit message: atlas control works

File: examples/valkyrie/urdf/atlas_urdf/atlas_convex_hull.urdf (robot description, URDF)
Before this commit: robot atlas, 70 links, 69 joints
Links:
- link l_clav: geometry collision mesh filename=package://valkyrie/urdf/meshes/r_clav_chull.obj; visual mesh filename=package://valkyrie/urdf/atlas)umeshes/r_clav.obj
